File: Hardware/Schematic.sch (EAGLE design)
At the start: 104 parts, among them IC1 BQ25180YBGR_BQ25180YBGR, IC2 DRV2605YZFR, IC3 BMA423, IC9 RT6160AWSC, J1 TC2030-IDC, J2 503480-2400, J4 KH-TYPE-C-16P, Q1 20V/4.2A/52mΩ/1.4W, Q3 SI1308EDL-T1-GE3, SW1 2025-10-22_07-23-44_LIBRARY_E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, SW2 2025-10-22_07-23-44_LIBRARY_E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, SW3 2025-10-22_07-23-44_LIBRARY_E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, U1 NRF52840_QF, U3 MAX17048G+T10, X1 32MHz, X2 32.768kHz

Commit message: Added files for review
Parts:
- removed C20: 4.7uF, InkTime_v5:NORDIC_NRF_3_CAPACITOR_0201_L
- removed D3: USBLC6-2SC6Y, InkTime_v5:ESP32_C6_LIBRARY_3_USBLC6-2SC6Y
- removed R1: 3K3, Resistor:R_CHIP-0402(1005-METRIC)
- removed R10, R11, R12, R6: (no value), Resistor:R_CHIP-0402(1005-METRIC)
- removed U$1, U$10, U$11, U$12, U$14, U$15, U$16, U$17, U$18, U$19, U$2, U$3, U$5, U$6, U$7, U$8, U$9: (no value), InkTime_v5:NORDIC_NRF_3_CAPACITOR_0201_L
- added C2-EP-DR: 4.7uF/25V, InkTime_v5:NORDIC_NRF_3_CAPACITOR_0402_L
- added C20\, C43: 4.7uF, InkTime_v5:NORDIC_NRF_3_CAPACITOR_0402_L
- added C27, C42: 0.1uF, InkTime_v5:NORDIC_NRF_3_CAPACITOR_0201_L
- added C29, C30, C31, C32: 1uF, InkTime_v5:NORDIC_NRF_3_CAPACITOR_0402_L
- added D1: USBLC6-2SC6Y, InkTime_v5:USBLC6-2SC6Y
- added EPD_C1, EPD_C10, EPD_C11, EPD_C12, EPD_C2, EPD_C6, EPD_C7, EPD_C8, EPD_C9: 1uF/50V, InkTime_v5:NORDIC_NRF_3_CAPACITOR_0402_L
- added R17, R18: 3K3, InkTime_v5:CPF0201D7K68C1_CPF0201D7K68C1
- added R1_USB, R2_USB: 5K1, InkTime_v5:CPF0201D7K68C1_CPF0201D7K68C1
- added R_PWR_EDP: 10K, InkTime_v5:CPF0201D7K68C1_CPF0201D7K68C1
- C1-EP-DR, C14, C15, C21, C24, C25, C33, C38, C6: device InkTime_v5:NORDIC_NRF_3_CAPACITOR_0201_L -> InkTime_v5:NORDIC_NRF_3_CAPACITOR_0402_L
- C34: value (none) -> 0.1uF
- C37, C39: device InkTime_v5:PERFECT_0402_CAP_0402 -> InkTime_v5:NORDIC_NRF_3_CAPACITOR_0402_L
- EPD_C5: value (none) -> 0.1uF/50V
- R1_EP_DR, R2, R2_EP_DR, R3, R4, R9, R_TYPE_SEL: device Resistor:R_CHIP-0402(1005-METRIC) -> InkTime_v5:CPF0201D7K68C1_CPF0201D7K68C1
- R5: value 3K3 -> 10K; device Resistor:R_CHIP-0402(1005-METRIC) -> InkTime_v5:CPF0201D7K68C1_CPF0201D7K68C1
- R7, R8: value (none) -> 10K; device Resistor:R_CHIP-0402(1005-METRIC) -> InkTime_v5:CPF0201D7K68C1_CPF0201D7K68C1
- renumbered U$13 to C34, U$4 to EPD_C5
Connections:
- removed net ALERT/1.6C: U3.!ALERT
- removed net ALERT/2.5C: U1.P0.10/NFC2@J24
- removed net D+/1.5D: D3.I/O2_2
- removed net D+/2.7D: U1.D+@AD6
- removed net D-/1.5D: D3.I/O1_2
- removed net D-/2.7D: U1.D-@AD4
- removed net EPD_BUSY/1.5D: J2.9
- removed net EPD_BUSY/2.2D: U1.P0.17@AD12
- removed net EPD_CS/1.5D: J2.12
- removed net EPD_CS/2.2D: U1.P0.05/AIN3@K2
- removed net EPD_DC/1.5D: J2.11
- removed net EPD_DC/2.2D: U1.P0.15@AD10
- removed net EPD_RST/1.5D: J2.10
- removed net EPD_RST/2.2D: U1.P0.16@AC11
- removed net HAPTIC_EN/1.4C: IC2.EN
- removed net HAPTIC_EN/2.6A: U1.P0.12@U1
- removed net MOSI/1.5D: J2.14
- removed net MOSI/2.2D: U1.P0.03/AIN1@B13
- removed net N$10: C12.2, U1.VDD@A22
- removed net N$18: Q3.S, R1_EP_DR.2
- removed net N$30: J4.SBU1
- removed net P0.13/1.5D: R10.1, SW2.2, U$14.1
- removed net P0.14/1.5D: R8.1, SW1.2, U$15.1
- removed net P0.14/2.7C: U1.P0.14@AC9
- removed net P1.01/1.6C: Q1.G, R6.1
- removed net P1.01/2.4B: U1.P1.01@Y23
- removed net P1.02/1.6C: R7.1, SW3.2, U$16.1
- removed net P1.02/2.8C: U1.P1.02@W24
- removed net PO.13/2.6C: U1.P0.13@AD8
- removed net SCK/1.5D: J2.13
- removed net SCK/2.2D: U1.P0.02/AIN0@A12
- new net ALERT: U1.P0.10/NFC2@J24, U3.!ALERT
- new net D+: D1.I/O2_2, U1.D+@AD6
- new net D-: D1.I/O1_2, U1.D-@AD4
- new net EPD_BUSY: J2.9, U1.P0.17@AD12
- new net EPD_CS: J2.12, U1.P0.05/AIN3@K2
- new net EPD_DC: J2.11, U1.P0.15@AD10
- new net EPD_RST: J2.10, U1.P0.16@AC11
- new net HAPTIC_EN: IC2.EN, U1.P0.12@U1
- new net MOSI: J2.14, U1.P0.03/AIN1@B13
- new net P0.13: C30.1, R5.1, SW2.2, U1.P0.13@AD8
- new net P0.14: C31.1, R8.1, SW1.2, U1.P0.14@AC9
- new net P1.01: Q1.G, R_PWR_EDP.1, U1.P1.01@Y23
- new net P1.02: C29.1, R7.1, SW3.2, U1.P1.02@W24
- new net SCK: J2.13, U1.P0.02/AIN0@A12
- net 3V3/1.7D: now also R5.2, R_PWR_EDP.2; no longer R10.2, R6.2
- net 3V3/2.4A: now also C12.2, C14.1, C25.1, C33.1, C6.1, R17.1, R18.1, U1.VDD@A22; no longer C14.2, C25.2, C33.2, C6.2, R1.1, R5.1
- net DN: now also D1.I/O1_1; no longer D3.I/O1_1
- net DP: now also D1.I/O2_1; no longer D3.I/O2_1
- net GND: now also C14.2, C15.2, C20\.2, C21.2, C25.2, C27.2, C29.2, C30.2, C31.2, C32.2, C33.2, C34.2, C38.2, C42.2, C43.2, C6.2, D1.GND, EPD_C1.1, EPD_C10.1, EPD_C11.1, EPD_C12.1, EPD_C2.1, EPD_C6.1, EPD_C7.1, EPD_C8.1, EPD_C9.1, R1_USB.1, R2_USB.2; no longer C14.1, C15.1, C20.1, C21.1, C25.1, C33.1, C38.1, C6.1, D3.GND, R11.1, R12.2, U$10.1, U$11.1, U$12.2, U$14.2, U$15.2, U$16.2, U$17.2, U$18.2, U$19.2, U$2.1, U$3.1, U$5.1, U$6.1, U$7.1, U$8.1, U$9.1
- net N$12: now also C15.1; no longer C15.2
- net N$15: now also C20\.1; no longer C20.2
- net N$19: now also C2-EP-DR.2; no longer U$1.2
- net N$21: now also C2-EP-DR.1; no longer U$1.1
- net N$22: now also EPD_C2.2; no longer U$3.2
- net N$23: now also EPD_C1.2; no longer U$2.2
- net N$24: now also C32.1; no longer U$12.1
- net N$25: now also EPD_C6.2; no longer U$9.2
- net N$26: now also EPD_C7.2; no longer U$7.2
- net N$27: now also EPD_C8.2; no longer U$11.2
- net N$28: now also R2_USB.1; no longer R12.1
- net N$29: now also EPD_C10.2; no longer U$10.2
- net N$31: now also EPD_C12.2; no longer U$8.2
- net N$34: now also R1_USB.2; no longer R11.2
- net PREVGH: now also EPD_C9.2; no longer U$5.2
- net PREVGL: now also EPD_C11.2; no longer U$6.2
- net RESE: now also Q3.S, R1_EP_DR.2
- net SCL/2.4C: now also R17.2; no longer R5.2
- net SDA/2.4C: now also R18.2; no longer R1.2
- net VBAT/1.2A: now also C27.1; no longer U$19.1
- net VBUS/1.5D: now also C42.1, C43.1, D1.VBUS; no longer D3.VBUS, U$17.1, U$18.1
- net VBUS/2.6D: now also C21.1, C38.1; no longer C21.2, C38.2
Other:
- note added: "Buttons"
- note added: "DC/DC"
- note added: "E-Paper Display Connector"
- note added: "E-Paper Drive Circuit"
- note added: "Fuel Gauge"
- note added: "Haptic Driver"
- note added: "IMU"
- note added: "LiPo Charger"
- note added: "SWD"
- note added: "USB C Connector & ESD Protection"
- moved on the sheet: C1-EP-DR, C14, C15, C21, C25, C33, C38, C6, D2, D4, D5, L5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

Commit message: Update Schematic.sch
Connections:
- removed net SCL/1.4C: IC2.SCL, U3.SCL
- removed net SDA/1.4C: IC2.SDA, U3.SDA
- removed net SDA/2.4C: IC1.SDA, IC3.SDX, R18.2, R2.2, TP_SDA.TP, U1.P0.06@L1
- removed net VBAT/1.2A: C27.1, TP_VBAT.TP, U3.CELL, U3.VDD
- removed net VBAT/2.5C: C37.1, IC1.BAT
- removed net VBUS/2.6D: C21.1, C38.1, IC1.IN, U1.VBUS@AD2
- new net SCL: IC1.SCL, IC2.SCL, U1.P0.07@M2, U3.SCL
- new net SDA: IC1.SDA, IC2.SDA, IC3.SDX, R18.2, R2.2, TP_SDA.TP, U1.P0.06@L1, U3.SDA
- new net VBAT: C27.1, C37.1, IC1.BAT, TP_VBAT.TP, U3.CELL, U3.VDD
- new net VBUS: C21.1, C38.1, D1.VBUS, IC1.IN, U1.VBUS@AD2
- net SCL/2.4C: no longer IC1.SCL, U1.P0.07@M2
- net VBUS/1.5D: no longer D1.VBUS
Other:
- moved on the sheet: C27, D1, TP_BA_GND, TP_VBAT, U3

Commit message: Update PCB
Parts:
- added C2: 12pF, InkTime_v5:NORDIC_NRF_3_CAPACITOR_0201_L
- EPD_C5: device InkTime_v5:NORDIC_NRF_3_CAPACITOR_0201_L -> InkTime_v5:NORDIC_NRF_3_CAPACITOR_0402_L
- renumbered TP_BA_GND to TP_BAT_GND
Connections:
- removed net 3V3/1.7D: C34.1, IC2.VDD, Q1.S, R5.2, R7.2, R8.2, R_PWR_EDP.2
- removed net 3V3/2.4A: C12.2, C14.1, C19.2, C25.1, C33.1, C6.1, C7.2, C8.2, IC3.CSB, IC3.VDD, IC3.VDDIO, IC9.VOUT_1, IC9.VOUT_2, J1.1, R17.1, R18.1, TP_3.3V.TP, TP_3V3.TP, U1.VDD@A22, U1.VDD@AD14, U1.VDD@AD23, U1.VDD@B1, U1.VDD@W1, U1.VDDH@Y2
- removed net P0.04: U1.P0.04/AIN2@J1
- removed net P0.09: U1.P0.09/NFC1@L24
- removed net P0.19: U1.P0.19@AC15
- removed net P0.20: U1.P0.20@AD16
- removed net P0.21: U1.P0.21@AC17
- removed net P0.22: U1.P0.22@AD18
- removed net P0.23: U1.P0.23@AC19
- removed net P0.24: U1.P0.24@AD20
- removed net P0.25: U1.P0.25@AC21
- removed net P0.26: U1.P0.26@G1
- removed net P0.27: U1.P0.27@H2
- removed net P0.28: U1.P0.28/AIN4@B11
- removed net P0.29: U1.P0.29/AIN5@A10
- removed net P0.30: U1.P0.30/AIN6@B9
- removed net P0.31: U1.P0.31/AIN7@A8
- removed net P1.03: U1.P1.03@V23
- removed net P1.04: U1.P1.04@U24
- removed net P1.05: U1.P1.05@T23
- removed net P1.06: U1.P1.06@R24
- removed net P1.07: U1.P1.07@P23
- removed net P1.09: U1.P1.09@R1
- removed net P1.10: U1.P1.10@A20
- removed net P1.11: U1.P1.11@B19
- removed net P1.12: U1.P1.12@B17
- removed net P1.13: U1.P1.13@A16
- removed net P1.14: U1.P1.14@B15
- removed net P1.15: U1.P1.15@A14
- removed net SCL/2.4C: IC3.SCX, R17.2, R4.2, TP_SCL.TP
- removed net VBUS/1.5D: C42.1, C43.1, J4.VBUS
- new net 3V3: C12.2, C14.1, C19.2, C25.1, C33.1, C34.1, C6.1, C7.2, C8.2, IC2.VDD, IC3.CSB, IC3.VDD, IC3.VDDIO, IC9.VOUT_1, IC9.VOUT_2, J1.1, Q1.S, R17.1, R18.1, R5.2, R7.2, R8.2, R_PWR_EDP.2, TP_3.3V.TP, TP_3V3.TP, U1.VDD@A22, U1.VDD@AD14, U1.VDD@AD23, U1.VDD@B1, U1.VDD@W1, U1.VDDH@Y2
- new net N$30: C2.1, U1.XC2@A23, X1.3
- net GND: now also C2.2; no longer U1.XC2@A23, X1.3
- net SCL: now also IC3.SCX, R17.2, R4.2, TP_SCL.TP
- net VBUS: now also C42.1, C43.1, J4.VBUS
Other:
- moved on the sheet: C19, IC3, R3

Commit message: Add PCB design, manufacturing files and docs
Parts:
- L2: device InkTime_v5:NORDIC_NRF_2_INDUCTOR_0402_L -> InkTime_v5:NORDIC_NRF_2_INDUCTOR_0603_L
Connections:
- net N$12 renamed DEC4_6
- net N$16 renamed DEC1
- net N$17 renamed P0.01/XL2
- net N$8 renamed DEC3
- net N$9 renamed P0.00/XL1
- removed net N$13: L2.2, L3.1
- new net N$8: L2.1, L3.1
- net N$14: now also L2.2; no longer L2.1
Other:
- moved on the sheet: L2
